File: Schematics/Relay Driver/Relay Driver_V1.1.brd (EAGLE design)
At the start: 76.2 x 50.8 mm, 16 parts

Commit message: updated berbers for relay driver
Parts:
- removed C1, C3: 470uF, rcl:E3,5-10
- added C5: 10uF, rcl:E3,5-10
- added D2: 5.1V, diode:DO35Z10
- added IC1: 74AC04N, 74xx-eu:DIL14
- added R5, R6: 1k, rcl:P0613V
- C2, C4: value 470uF -> 4.7uF
- moved R1 12.8 mm to (33.0, 24.1)
- moved R3 12.7 mm to (33.0, 27.9)
- moved T2 10.2 mm to (36.8, 31.8)
- moved T1 10.2 mm to (39.4, 20.3)
- moved R2 5.08 mm to (15.2, 10.2)
- moved LED1 4.58 mm to (26.7, 11.4)
- moved LED2 2.54 mm to (26.7, 35.6)
- moved C4 2.54 mm to (22.9, 44.5), turned to 270 degrees
- moved R4 1.27 mm to (15.2, 36.8)
Connections:
- new net N$12: C5.+, IC1.14, R6.2
- new net N$13: D2.C, R5.2, R6.1
- new net N$6: IC1.1, U$1.2
- new net N$8: IC1.3, U$1.3
- net +8V: now also R5.1
- net G0: now also IC1.2; no longer U$1.2
- net G1: now also IC1.4; no longer U$1.3
- net GND: now also C5.-, D2.A, IC1.7; no longer C1.-, C3.-
- net N$1: no longer C1.+
- net N$3: no longer C3.+
Routing:
- net G0: track 13.2 -> 42.0 mm
- net G1: track 13.2 -> 36.4 mm
- net N$12: track 0.00 -> 17.3 mm
- net N$6: track 0.00 -> 9.94 mm
- net N$3: track 14.0 -> 5.61 mm
- net N$1: track 14.0 -> 5.61 mm
- net N$13: track 0.00 -> 7.62 mm
- net N$8: track 0.00 -> 7.40 mm
- net N$7: track 15.8 -> 21.7 mm
- net N$9: track 5.08 -> 8.15 mm
- net N$10: track 5.08 -> 8.15 mm
- net +8V: track 123.8 -> 121.0 mm
- net N$4: track 59.1 -> 56.5 mm
