File: Schematics/Relay Driver/Relay Driver_V1.1.sch (EAGLE design)
At the start: 16 parts

Commit message: updated berbers for relay driver
Parts:
- removed C1, C3: 470uF, rcl:CPOL-EUE3.5-10
- added C5: 10uF, rcl:CPOL-EUE3.5-10
- added D2: 5.1V, diode:ZENER-DIODEDO35Z10
- added IC1: 74AC04N, 74xx-eu:74AC04N
- added R5, R6: 1k, rcl:R-US_0613/5V
- C2, C4: value 470uF -> 4.7uF
Connections:
- new net N$12: C5.+, IC1P.VCC, R6.2
- new net N$13: D2.C, R5.2, R6.1
- new net N$6: IC1A.I, U$1.2
- new net N$8: IC1B.I, U$1.3
- net +8V: now also R5.1
- net G0: now also IC1A.O; no longer U$1.2
- net G1: now also IC1B.O; no longer U$1.3
- net GND: now also C5.-, D2.A, IC1P.GND; no longer C1.-, C3.-
- net N$1: no longer C1.+
- net N$3: no longer C3.+
Changed lines of the file:
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@@
 <part name="R1" library="rcl" deviceset="R-US_" device="0613/5V" value="1k"/>
 <part name="D1" library="diode" deviceset="1N4148" device="DO35-10"/>
-<part name="C1" library="rcl" deviceset="CPOL-EU" device="E3.5-10" value="470uF"/>
-<part name="C2" library="rcl" deviceset="CPOL-EU" device="E3.5-10" value="470uF"/>
-<part name="GND1" library="supply1" deviceset="GND" device=""/>
+<part name="C2" library="rcl" deviceset="CPOL-EU" device="E3.5-10" value="4.7uF"/>
 <part name="GND2" library="supply1" deviceset="GND" device=""/>
 <part name="U$2" library="Headers" deviceset="1X2HEADER_100MIL" device=""/>
@@
 <part name="T2" library="transistor" deviceset="*-NPN-" device="TO92-EBC"/>
 <part name="R3" library="rcl" deviceset="R-US_" device="0613/5V" value="1k"/>
-<part name="C3" library="rcl" deviceset="CPOL-EU" device="E3.5-10" value="470uF"/>
-<part name="C4" library="rcl" deviceset="CPOL-EU" device="E3.5-10" value="470uF"/>
-<part name="GND4" library="supply1" deviceset="GND" device=""/>
+<part name="C4" library="rcl" deviceset="CPOL-EU" device="E3.5-10" value="4.7uF"/>
 <part name="GND5" library="supply1" deviceset="GND" device=""/>
 <part name="R4" library="rcl" deviceset="R-US_" device="0613/5V" value="1k"/>
@@
 <part name="SUPPLY3" library="supply2" deviceset="+8V" device=""/>
 <part name="RL1" library="relay" deviceset="FRL-264" device=""/>
+<part name="IC1" library="74xx-eu" deviceset="74*04" device="N" technology="AC"/>
+<part name="D2" library="diode" deviceset="ZENER-DIODE" device="DO35Z10" value="5.1V"/>
+<part name="R5" library="rcl" deviceset="R-US_" device="0613/5V" value="1k"/>
+<part name="R6" library="rcl" deviceset="R-US_" device="0613/5V" value="1k"/>
+<part name="C5" library="rcl" deviceset="CPOL-EU" device="E3.5-10" value="10uF"/>
+<part name="SUPPLY4" library="supply2" deviceset="+8V" device=""/>
+<part name="GND6" library="supply1" deviceset="GND" device=""/>
+<part name="GND7" library="supply1" deviceset="GND" device=""/>
+<part name="GND8" library="supply1" deviceset="GND" device=""/>
 </parts>
 <sheets>
@@
 <instance part="R1" gate="G$1" x="132.08" y="68.58"/>
 <instance part="D1" gate="G$1" x="142.24" y="88.9" rot="R90"/>
-<instance part="C1" gate="G$1" x="139.7" y="60.96"/>
 <instance part="C2" gate="G$1" x="132.08" y="88.9"/>
-<instance part="GND1" gate="1" x="139.7" y="50.8"/>
 <instance part="GND2" gate="1" x="149.86" y="50.8"/>
 <instance part="U$2" gate="G$1" x="200.66" y="93.98" rot="R180"/>
@@
 <instance part="T2" gate="G$1" x="134.62" y="134.62"/>
 <instance part="R3" gate="G$1" x="119.38" y="134.62"/>
-<instance part="C3" gate="G$1" x="127" y="127"/>
 <instance part="C4" gate="G$1" x="119.38" y="154.94"/>
-<instance part="GND4" gate="1" x="127" y="116.84"/>
 <instance part="GND5" gate="1" x="137.16" y="116.84"/>
 <instance part="R4" gate="G$1" x="137.16" y="162.56" rot="R90"/>
@@
 <instance part="RL1" gate="G$2" x="167.64" y="86.36"/>
 <instance part="RL1" gate="G$3" x="167.64" y="104.14"/>
+<instance part="IC1" gate="A" x="73.66" y="93.98"/>
+<instance part="IC1" gate="B" x="73.66" y="81.28"/>
+<instance part="IC1" gate="P" x="48.26" y="152.4"/>
+<instance part="D2" gate="G$1" x="71.12" y="152.4" rot="R90"/>
+<instance part="R5" gate="G$1" x="83.82" y="165.1" rot="R180"/>
+<instance part="R6" gate="G$1" x="60.96" y="165.1" rot="R180"/>
+<instance part="C5" gate="G$1" x="38.1" y="154.94"/>
+<instance part="SUPPLY4" gate="+8V" x="88.9" y="172.72"/>
+<instance part="GND6" gate="1" x="48.26" y="139.7"/>
+<instance part="GND7" gate="1" x="38.1" y="139.7"/>
+<instance part="GND8" gate="1" x="71.12" y="139.7"/>
 </instances>
 <busses>
@@
 <pinref part="R1" gate="G$1" pin="2"/>
 <pinref part="T1" gate="G$1" pin="B"/>
-<wire x1="137.16" y1="68.58" x2="139.7" y2="68.58" width="0.1524" layer="91"/>
-<pinref part="C1" gate="G$1" pin="+"/>
-<wire x1="139.7" y1="68.58" x2="144.78" y2="68.58" width="0.1524" layer="91"/>
-<wire x1="139.7" y1="63.5" x2="139.7" y2="68.58" width="0.1524" layer="91"/>
-<junction x="139.7" y="68.58"/>
+<wire x1="137.16" y1="68.58" x2="144.78" y2="68.58" width="0.1524" layer="91"/>
 </segment>
 </net>
@@
 <pinref part="R1" gate="G$1" pin="1"/>
 <wire x1="127" y1="68.58" x2="83.82" y2="68.58" width="0.1524" layer="91"/>
-<wire x1="48.26" y1="86.36" x2="83.82" y2="86.36" width="0.1524" layer="91"/>
-<wire x1="83.82" y1="86.36" x2="83.82" y2="68.58" width="0.1524" layer="91"/>
-<pinref part="U$1" gate="G$1" pin="3"/>
-<label x="68.58" y="86.36" size="1.778" layer="95"/>
+<label x="88.9" y="81.28" size="1.778" layer="95"/>
+<pinref part="IC1" gate="B" pin="O"/>
+<wire x1="83.82" y1="81.28" x2="83.82" y2="68.58" width="0.1524" layer="91"/>
 </segment>
 </net>
 <net name="GND" class="0">
-<segment>
-<pinref part="C1" gate="G$1" pin="-"/>
-<pinref part="GND1" gate="1" pin="GND"/>
-<wire x1="139.7" y1="55.88" x2="139.7" y2="53.34" width="0.1524" layer="91"/>
-</segment>
 <segment>
 <pinref part="T1" gate="G$1" pin="E"/>
@@
 </segment>
 <segment>
-<pinref part="C3" gate="G$1" pin="-"/>
-<pinref part="GND4" gate="1" pin="GND"/>
-<wire x1="127" y1="121.92" x2="127" y2="119.38" width="0.1524" layer="91"/>
-</segment>
-<segment>
 <pinref part="T2" gate="G$1" pin="E"/>
 <wire x1="137.16" y1="129.54" x2="137.16" y2="119.38" width="0.1524" layer="91"/>
 <pinref part="GND5" gate="1" pin="GND"/>
+</segment>
+<segment>
+<pinref part="C5" gate="G$1" pin="-"/>
+<pinref part="GND7" gate="1" pin="GND"/>
+<wire x1="38.1" y1="149.86" x2="38.1" y2="142.24" width="0.1524" layer="91"/>
+</segment>
+<segment>
+<pinref part="D2" gate="G$1" pin="A"/>
+<pinref part="GND8" gate="1" pin="GND"/>
+<wire x1="71.12" y1="149.86" x2="71.12" y2="142.24" width="0.1524" layer="91"/>
+</segment>
+<segment>
+<pinref part="IC1" gate="P" pin="GND"/>
+<pinref part="GND6" gate="1" pin="GND"/>
+<wire x1="48.26" y1="144.78" x2="48.26" y2="142.24" width="0.1524" layer="91"/>
 </segment>
 </net>
@@
 <pinref part="R3" gate="G$1" pin="2"/>
 <pinref part="T2" gate="G$1" pin="B"/>
-<wire x1="124.46" y1="134.62" x2="127" y2="134.62" width="0.1524" layer="91"/>
-<pinref part="C3" gate="G$1" pin="+"/>
-<wire x1="127" y1="134.62" x2="132.08" y2="134.62" width="0.1524" layer="91"/>
-<wire x1="127" y1="129.54" x2="127" y2="134.62" width="0.1524" layer="91"/>
-<junction x="127" y="134.62"/>
+<wire x1="124.46" y1="134.62" x2="132.08" y2="134.62" width="0.1524" layer="91"/>
 </segment>
 </net>
@@
 <net name="G0" class="0">
 <segment>
-<pinref part="U$1" gate="G$1" pin="2"/>
-<wire x1="48.26" y1="88.9" x2="83.82" y2="88.9" width="0.1524" layer="91"/>
-<wire x1="83.82" y1="88.9" x2="83.82" y2="134.62" width="0.1524" layer="91"/>
 <pinref part="R3" gate="G$1" pin="1"/>
+<wire x1="83.82" y1="93.98" x2="83.82" y2="134.62" width="0.1524" layer="91"/>
 <wire x1="83.82" y1="134.62" x2="114.3" y2="134.62" width="0.1524" layer="91"/>
-<label x="68.58" y="88.9" size="1.778" layer="95"/>
+<label x="88.9" y="101.6" size="1.778" layer="95"/>
+<pinref part="IC1" gate="A" pin="O"/>
 </segment>
 </net>
@@
 <junction x="137.16" y="167.64"/>
 </segment>
+<segment>
+<pinref part="R5" gate="G$1" pin="1"/>
+<wire x1="88.9" y1="165.1" x2="88.9" y2="170.18" width="0.1524" layer="91"/>
+<pinref part="SUPPLY4" gate="+8V" pin="+8V"/>
+</segment>
 </net>
 <net name="N$2" class="0">
@@
 </segment>
 </net>
+<net name="N$6" class="0">
+<segment>
+<pinref part="U$1" gate="G$1" pin="2"/>
+<wire x1="48.26" y1="88.9" x2="58.42" y2="88.9" width="0.1524" layer="91"/>
+<wire x1="58.42" y1="88.9" x2="58.42" y2="93.98" width="0.1524" layer="91"/>
+<pinref part="IC1" gate="A" pin="I"/>
+<wire x1="58.42" y1="93.98" x2="63.5" y2="93.98" width="0.1524" layer="91"/>
+</segment>
+</net>
+<net name="N$8" class="0">
+<segment>
+<pinref part="IC1" gate="B" pin="I"/>
+<wire x1="63.5" y1="81.28" x2="58.42" y2="81.28" width="0.1524" layer="91"/>
+<wire x1="58.42" y1="81.28" x2="58.42" y2="86.36" width="0.1524" layer="91"/>
+<pinref part="U$1" gate="G$1" pin="3"/>
+<wire x1="58.42" y1="86.36" x2="48.26" y2="86.36" width="0.1524" layer="91"/>
+</segment>
+</net>
+<net name="N$12" class="0">
+<segment>
+<pinref part="C5" gate="G$1" pin="+"/>
+<wire x1="38.1" y1="157.48" x2="38.1" y2="165.1" width="0.1524" layer="91"/>
+<pinref part="IC1" gate="P" pin="VCC"/>
+<wire x1="38.1" y1="165.1" x2="48.26" y2="165.1" width="0.1524" layer="91"/>
+<wire x1="48.26" y1="165.1" x2="48.26" y2="160.02" width="0.1524" layer="91"/>
+<pinref part="R6" gate="G$1" pin="2"/>
+<wire x1="55.88" y1="165.1" x2="48.26" y2="165.1" width="0.1524" layer="91"/>
+<junction x="48.26" y="165.1"/>
+</segment>
+</net>
+<net name="N$13" class="0">
+<segment>
+<pinref part="R6" gate="G$1" pin="1"/>
+<pinref part="R5" gate="G$1" pin="2"/>
+<wire x1="66.04" y1="165.1" x2="71.12" y2="165.1" width="0.1524" layer="91"/>
+<pinref part="D2" gate="G$1" pin="C"/>
+<wire x1="71.12" y1="165.1" x2="78.74" y2="165.1" width="0.1524" layer="91"/>
+<wire x1="71.12" y1="154.94" x2="71.12" y2="165.1" width="0.1524" layer="91"/>
+<junction x="71.12" y="165.1"/>
+</segment>
+</net>
